File: lab4/lab4 exercise 1/lab4 exercise 1.kicad_sch (KiCad schematic)
At the start: 6 parts, among them SW1 SW_SPDT

Commit message: lab6 done
Parts:
- C1: footprint (none) -> Capacitor_THT:C_Radial_D5.0mm_H5.0mm_P2.00mm
- D1: footprint (none) -> LED_THT:LED_D5.0mm
- R1, R2: footprint (none) -> Resistor_THT:R_Axial_DIN0516_L15.5mm_D5.0mm_P20.32mm_Horizontal
- SW1: footprint (none) -> Button_Switch_THT:SW_E-Switch_EG1224_SPDT_Angled
- V1: footprint (none) -> Connector_JST:JST_PH_B2B-PH-K_1x02_P2.00mm_Vertical
Changed lines of the file:
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@@
       (effects (font (size 1.27 1.27)) (justify right) hide)
     )
-    (property "Footprint" "" (id 2) (at 166.37 104.14 0)
-      (effects (font (size 1.27 1.27)) hide)
-    )
+    (property "Footprint" "LED_THT:LED_D5.0mm" (id 2) (at 179.07 104.14 90))
     (property "Datasheet" "~" (id 3) (at 166.37 104.14 0)
       (effects (font (size 1.27 1.27)) hide)
@@
   )
   (symbol (lib_id "Device:C_Polarized") (at 148.59 100.33 0) (unit 1)
-    (in_bom yes) (on_board yes) (fields_autoplaced)
+    (in_bom yes) (on_board yes)
     (property "Reference" "C1" (id 0) (at 152.4 98.1709 0)
       (effects (font (size 1.27 1.27)) (justify left))
@@
       (effects (font (size 1.27 1.27)) (justify left))
     )
-    (property "Footprint" "" (id 2) (at 149.5552 104.14 0)
-      (effects (font (size 1.27 1.27)) hide)
-    )
+    (property "Footprint" "Capacitor_THT:C_Radial_D5.0mm_H5.0mm_P2.00mm" (id 2) (at 134.62 104.14 0))
     (property "Datasheet" "~" (id 3) (at 148.59 100.33 0)
       (effects (font (size 1.27 1.27)) hide)
@@
     (property "Reference" "R2" (id 0) (at 133.35 93.98 90))
     (property "Value" "2.2 kΩ" (id 1) (at 133.35 96.52 90))
-    (property "Footprint" "" (id 2) (at 133.35 93.218 90)
-      (effects (font (size 1.27 1.27)) hide)
-    )
+    (property "Footprint" "Resistor_THT:R_Axial_DIN0516_L15.5mm_D5.0mm_P20.32mm_Horizontal" (id 2) (at 101.6 88.9 90))
     (property "Datasheet" "~" (id 3) (at 133.35 91.44 0)
       (effects (font (size 1.27 1.27)) hide)
@@
       (effects (font (size 1.27 1.27)) hide)
     )
-    (property "Footprint" "" (id 2) (at 142.24 91.44 0)
-      (effects (font (size 1.27 1.27)) hide)
-    )
+    (property "Footprint" "Button_Switch_THT:SW_E-Switch_EG1224_SPDT_Angled" (id 2) (at 151.13 85.09 0))
     (property "Datasheet" "~" (id 3) (at 142.24 91.44 0)
       (effects (font (size 1.27 1.27)) hide)
@@
   )
   (symbol (lib_id "Device:R") (at 166.37 95.25 180) (unit 1)
-    (in_bom yes) (on_board yes) (fields_autoplaced)
+    (in_bom yes) (on_board yes)
     (property "Reference" "R1" (id 0) (at 168.91 93.9799 0)
       (effects (font (size 1.27 1.27)) (justify right))
@@
       (effects (font (size 1.27 1.27)) (justify right))
     )
-    (property "Footprint" "" (id 2) (at 168.148 95.25 90)
-      (effects (font (size 1.27 1.27)) hide)
-    )
+    (property "Footprint" "Resistor_THT:R_Axial_DIN0516_L15.5mm_D5.0mm_P20.32mm_Horizontal" (id 2) (at 194.31 88.9 0))
     (property "Datasheet" "~" (id 3) (at 166.37 95.25 0)
       (effects (font (size 1.27 1.27)) hide)
@@
     (property "Reference" "V1" (id 0) (at 129.54 99.06 0))
     (property "Value" "9 V" (id 1) (at 129.54 101.6 0))
-    (property "Footprint" "" (id 2) (at 121.92 99.06 0)
-      (effects (font (size 1.27 1.27)) hide)
-    )
+    (property "Footprint" "Connector_JST:JST_PH_B2B-PH-K_1x02_P2.00mm_Vertical" (id 2) (at 95.25 95.25 0))
     (property "Datasheet" "~" (id 3) (at 121.92 99.06 0)
       (effects (font (size 1.27 1.27)) hide)
@@
   (symbol_instances
     (path "/856e2714-5c53-478c-95e4-4147c0f19b54"
-      (reference "C1") (unit 1) (value "4.7μF") (footprint "")
+      (reference "C1") (unit 1) (value "4.7μF") (footprint "Capacitor_THT:C_Radial_D5.0mm_H5.0mm_P2.00mm")
     )
     (path "/0f97689d-2572-45ce-825f-4aed20485a28"
-      (reference "D1") (unit 1) (value "LED") (footprint "")
+      (reference "D1") (unit 1) (value "LED") (footprint "LED_THT:LED_D5.0mm")
     )
     (path "/ec3c92b7-e706-415c-9f5e-1b79de1ada3a"
-      (reference "R1") (unit 1) (value "20 kΩ") (footprint "")
+      (reference "R1") (unit 1) (value "20 kΩ") (footprint "Resistor_THT:R_Axial_DIN0516_L15.5mm_D5.0mm_P20.32mm_Horizontal")
     )
     (path "/a6ce5810-137b-4e10-8bf8-6c5e7733960f"
-      (reference "R2") (unit 1) (value "2.2 kΩ") (footprint "")
+      (reference "R2") (unit 1) (value "2.2 kΩ") (footprint "Resistor_THT:R_Axial_DIN0516_L15.5mm_D5.0mm_P20.32mm_Horizontal")
     )
     (path "/bb21db69-e922-4adc-9f55-149161fe6458"
-      (reference "SW1") (unit 1) (value "SW_SPDT") (footprint "")
+      (reference "SW1") (unit 1) (value "SW_SPDT") (footprint "Button_Switch_THT:SW_E-Switch_EG1224_SPDT_Angled")
     )
     (path "/f1d93530-3fac-44ae-8d69-fb644a496ff5"
-      (reference "V1") (unit 1) (value "9 V") (footprint "")
+      (reference "V1") (unit 1) (value "9 V") (footprint "Connector_JST:JST_PH_B2B-PH-K_1x02_P2.00mm_Vertical")
     )
   )
